Commit message: Cập nhật code anviet_688 chuẩn chỉnh từ máy tính

File: description/robot.urdf.xacro (robot description, xacro)
@@ -1,4 +1,15 @@
 <?xml version="1.0"?>
-<robot xmlns:xacro="http://www.ros.org/wiki/xacro"  name="robot">
+<robot name="anviet_688" xmlns:xacro="http://www.ros.org/wiki/xacro">
+    <xacro:arg name="use_ros2_control" default="true"/>
     <xacro:include filename="robot_core.xacro" />
+    <!-- Switch between ros2_control and Gazebo integrated diff-drive control -->
+    <xacro:if value="$(arg use_ros2_control)">
+        <xacro:include filename="ros2_control.xacro" />
+    </xacro:if>
+    <xacro:unless value="$(arg use_ros2_control)">
+        <xacro:include filename="gazebo_control.xacro" />
+    </xacro:unless>
+    <xacro:include filename="gazebo_control.xacro" />
+    <xacro:include filename="lidar.xacro" />
+    <xacro:include filename="ros2_control.xacro"/>
 </robot>

File: description/robot_core.xacro (robot description, xacro)
@@ -14,4 +14,7 @@
         <color rgba="0 0 0 1"/>
     </material>
+    <material name="red">
+        <color rgba="1 0 0 1"/>
+    </material>
  <!--base link -->
     <link name="base_link">
@@ -21,22 +24,22 @@
         <parent link="base_link"/>
         <child link="chassis"/>
-        <origin xyz="-0.1 0 0"/>
+        <origin xyz="-0.03 0 0"/>
     </joint>
     <link name="chassis">
         <visual>
-            <origin xyz="0.15 0 0.075" rpy="0 0 0"/>
+            <origin xyz="0.105 0 0.03" rpy="0 0 0"/>
             <geometry>
-                <box size="0.21 0.15 0.15"/>
+                <box size="0.21 0.15 0.07"/>
             </geometry>
-            <material name="white"/>
+            <material name="black"/>
         </visual>
         <collision>
-            <origin xyz="0.15 0 0.075" rpy="0 0 0"/>
+            <origin xyz="0.105 0 0.03" rpy="0 0 0"/>
             <geometry>
-                <box size="0.21 0.15 0.15"/>
+                <box size="0.21 0.15 0.07"/>
             </geometry>
         </collision>
-        <xacro:inertial_box mass="0.5" x="0.21" y="0.15" z="0.15">
-            <origin xyz="0.15 0 0.075" rpy="0 0 0"/>
+        <xacro:inertial_box mass="0.5" x="0.21" y="0.15" z="0.07">
+            <origin xyz="0.15 0 0.03" rpy="0 0 0"/>
         </xacro:inertial_box>
     </link>
@@ -45,11 +48,12 @@
         <parent link="base_link"/>
         <child link="left_wheel"/>
-        <origin xyz="0 0.105 0" rpy="-${pi/2} 0 0"/>
+        <origin xyz="0 0.1025 -0.025" rpy="-${pi/2} 0 0"/>
         <axis xyz="0 0 1"/>
+        <limit effort="0.5" velocity="11.516"/>
     </joint>
     <link name="left_wheel">
         <visual>
             <geometry>
-                <cylinder length="0.04" radius="0.05" />
+                <cylinder length="0.025" radius="0.034" />
             </geometry>
             <material name="blue"/>
@@ -57,8 +61,8 @@
         <collision>
             <geometry>
-                <cylinder length="0.04" radius="0.05" />
+              <sphere radius="0.034" />
             </geometry>
         </collision>
-        <xacro:inertial_cylinder mass="0.1" length="0.04" radius="0.05">
+        <xacro:inertial_cylinder mass="0.1" length="0.025" radius="0.034">
             <origin xyz="0 0 0" rpy="0 0 0"/>
         </xacro:inertial_cylinder>
@@ -66,13 +70,14 @@
     <!-- RIGHT WHEEL -->
     <joint name="right_wheel_joint" type="continuous">
-        <parent link="base_link"/>
+       <parent link="base_link"/>
         <child link="right_wheel"/>
-        <origin xyz="0 -0.105 0" rpy="${pi/2} 0 0"/>
+        <origin xyz="0 -0.1025 -0.025" rpy="${pi/2} 0 0"/>
         <axis xyz="0 0 -1"/>
+        <limit effort="0.5" velocity="11.516"/>
     </joint>
     <link name="right_wheel">
         <visual>
             <geometry>
-                <cylinder length="0.04" radius="0.05" />
+                <cylinder length="0.025" radius="0.034" />
             </geometry>
             <material name="blue"/>
@@ -80,8 +85,8 @@
         <collision>
             <geometry>
-                <cylinder length="0.04" radius="0.05" />
+               <sphere radius="0.034" />
             </geometry>
         </collision>
-        <xacro:inertial_cylinder mass="0.1" length="0.04" radius="0.05">
+        <xacro:inertial_cylinder mass="0.1" length="0.025" radius="0.034">
             <origin xyz="0 0 0" rpy="0 0 0"/>
         </xacro:inertial_cylinder>
@@ -91,21 +96,25 @@
         <parent link="chassis"/>
         <child link="caster_wheel"/>
-        <origin xyz="0.2 0 0" rpy="0 0 0"/>
+        <origin xyz="0.175 0 -0.025" rpy="0 0 0"/>
     </joint>
     <link name="caster_wheel">
         <visual>
             <geometry>
-                <sphere radius="0.05" />
+                <sphere radius="0.034" />
             </geometry>
-            <material name="black"/>
+            <material name="white"/>
         </visual>
         <collision>
             <geometry>
-                <sphere radius="0.05" />
+                <sphere radius="0.034" />
             </geometry>
         </collision>
-        <xacro:inertial_sphere mass="0.1" radius="0.05">
+        <xacro:inertial_sphere mass="0.1" radius="0.034">
             <origin xyz="0 0 0" rpy="0 0 0"/>
         </xacro:inertial_sphere>
     </link>
+    <gazebo reference="caster_wheel">
+        <mu1 value="0.0"/>
+        <mu2 value="0.0"/>
+    </gazebo>
 </robot>
